File: esp8266/reader/esp8266RFIDReader.sch (KiCad schematic (older format))
At the start: 17 parts, among them J1 Conn_01x02, J2 Conn_01x05, U1 RFID_MODULE_125_KHZ

Commit message: Schematic and PCB for RFID control module.
Parts:
- D1, D2, D3, D4, D5: footprint LEDs:LED_1206_HandSoldering -> LEDs:LED_0603_HandSoldering
- R1, R2, R3, R4, R5, R6, R7: footprint Resistors_SMD:R_1206_HandSoldering -> Resistors_SMD:R_0805_HandSoldering
Changed lines of the file:
@@
 F 0 "R3" V 4680 3600 50  0000 C CNN
 F 1 "20k" V 4600 3600 50  0000 C CNN
-F 2 "Resistors_SMD:R_1206_HandSoldering" V 4530 3600 50  0001 C CNN
+F 2 "Resistors_SMD:R_0805_HandSoldering" V 4530 3600 50  0001 C CNN
 F 3 "" H 4600 3600 50  0001 C CNN
 	1    4600 3600
@@
 F 0 "R1" V 4430 3450 50  0000 C CNN
 F 1 "10k" V 4350 3450 50  0000 C CNN
-F 2 "Resistors_SMD:R_1206_HandSoldering" V 4280 3450 50  0001 C CNN
+F 2 "Resistors_SMD:R_0805_HandSoldering" V 4280 3450 50  0001 C CNN
 F 3 "" H 4350 3450 50  0001 C CNN
 	1    4350 3450
@@
 F 0 "R6" V 7530 3600 50  0000 C CNN
 F 1 "1k" V 7450 3600 50  0000 C CNN
-F 2 "Resistors_SMD:R_1206_HandSoldering" V 7380 3600 50  0001 C CNN
+F 2 "Resistors_SMD:R_0805_HandSoldering" V 7380 3600 50  0001 C CNN
 F 3 "" H 7450 3600 50  0001 C CNN
 	1    7450 3600
@@
 F 0 "R7" V 7530 3900 50  0000 C CNN
 F 1 "1k" V 7450 3900 50  0000 C CNN
-F 2 "Resistors_SMD:R_1206_HandSoldering" V 7380 3900 50  0001 C CNN
+F 2 "Resistors_SMD:R_0805_HandSoldering" V 7380 3900 50  0001 C CNN
 F 3 "" H 7450 3900 50  0001 C CNN
 	1    7450 3900
@@
 F 0 "D3" H 7850 3700 50  0000 C CNN
 F 1 "LED_B" H 7850 3500 50  0000 C CNN
-F 2 "LEDs:LED_1206_HandSoldering" H 7850 3600 50  0001 C CNN
+F 2 "LEDs:LED_0603_HandSoldering" H 7850 3600 50  0001 C CNN
 F 3 "" H 7850 3600 50  0001 C CNN
 	1    7850 3600
@@
 F 0 "D4" H 7850 4000 50  0000 C CNN
 F 1 "LED_Y" H 7850 3800 50  0000 C CNN
-F 2 "LEDs:LED_1206_HandSoldering" H 7850 3900 50  0001 C CNN
+F 2 "LEDs:LED_0603_HandSoldering" H 7850 3900 50  0001 C CNN
 F 3 "" H 7850 3900 50  0001 C CNN
 	1    7850 3900
@@
 F 0 "R2" V 4530 2300 50  0000 C CNN
 F 1 "1k" V 4450 2300 50  0000 C CNN
-F 2 "Resistors_SMD:R_1206_HandSoldering" V 4380 2300 50  0001 C CNN
+F 2 "Resistors_SMD:R_0805_HandSoldering" V 4380 2300 50  0001 C CNN
 F 3 "" H 4450 2300 50  0001 C CNN
 	1    4450 2300
@@
 F 0 "R5" V 6530 2750 50  0000 C CNN
 F 1 "1k" V 6450 2750 50  0000 C CNN
-F 2 "Resistors_SMD:R_1206_HandSoldering" V 6380 2750 50  0001 C CNN
+F 2 "Resistors_SMD:R_0805_HandSoldering" V 6380 2750 50  0001 C CNN
 F 3 "" H 6450 2750 50  0001 C CNN
 	1    6450 2750
@@
 F 0 "D2" H 6950 2850 50  0000 C CNN
 F 1 "LED_R" H 6950 2650 50  0000 C CNN
-F 2 "LEDs:LED_1206_HandSoldering" H 6950 2750 50  0001 C CNN
+F 2 "LEDs:LED_0603_HandSoldering" H 6950 2750 50  0001 C CNN
 F 3 "" H 6950 2750 50  0001 C CNN
 	1    6950 2750
@@
 F 0 "R4" V 6530 2350 50  0000 C CNN
 F 1 "1k" V 6450 2350 50  0000 C CNN
-F 2 "Resistors_SMD:R_1206_HandSoldering" V 6380 2350 50  0001 C CNN
+F 2 "Resistors_SMD:R_0805_HandSoldering" V 6380 2350 50  0001 C CNN
 F 3 "" H 6450 2350 50  0001 C CNN
 	1    6450 2350
@@
 F 0 "D1" H 6950 2450 50  0000 C CNN
 F 1 "LED_G" H 6950 2250 50  0000 C CNN
-F 2 "LEDs:LED_1206_HandSoldering" H 6950 2350 50  0001 C CNN
+F 2 "LEDs:LED_0603_HandSoldering" H 6950 2350 50  0001 C CNN
 F 3 "" H 6950 2350 50  0001 C CNN
 	1    6950 2350
@@
 F 0 "D5" H 7300 2850 50  0000 C CNN
 F 1 "LED_R" H 7300 2650 50  0000 C CNN
-F 2 "LEDs:LED_1206_HandSoldering" H 7300 2750 50  0001 C CNN
+F 2 "LEDs:LED_0603_HandSoldering" H 7300 2750 50  0001 C CNN
 F 3 "" H 7300 2750 50  0001 C CNN
 	1    7300 2750
